File: Hardware/PCB.brd (EAGLE design)
At the start: 170.2 x 111.2 mm, 103 parts, among them IC1 BD5229G-TR, IC4 XC6220A331MR-G, J1 FH34SRJ-24S-0.5SH_99_, J2 SAMACSYS_PARTS_USB4110-GF-A, J3 QWIIC_RIGHT_ANGLE, J4 112A-TAAR-R03_ATTEND, Q1 20V/4.2A/52mΩ/1.4W, Q2 20V/4.2A/52mΩ/1.4W, Q3 SI1308EDL-T1-GE3, U1 W25Q512JVEIQ, U2 ESP32-C6-WROOM-1-N8, U3 DS3231SN#, U4 MAX17048G+T10

Commit message: Fixed issues
Parts:
- moved R1_PWRUSB 8.60 mm to (119.1, 46.6), turned to 270 degrees
- moved BOOT_BUTTON 0.08 mm to (49.0, 108.8)
- moved CHANGE_BUTTON 0.08 mm to (64.0, 108.8)
- moved RESET_BUTTON 0.08 mm to (24.0, 108.8)
Routing:
- net GND: track 17773.0 -> 10.5 mm, vias 179 -> 95
- net 3V3: track 422.0 -> 446.9 mm
- net VBUS: track 197.2 -> 177.5 mm, vias 2 -> 4
- net EPD_DC: track 97.7 -> 117.1 mm
- net N$9: track 17.8 -> 31.5 mm, vias 2 -> 0
- net N$7: track 33.7 -> 41.6 mm
- net MOSI: track 180.1 -> 187.1 mm, vias 5 -> 6
- net FLASH_CS: track 47.0 -> 53.4 mm
- net EPD_3V3_C: track 124.8 -> 118.6 mm, vias 3 -> 6
- net N$19: track 17.9 -> 23.1 mm
- net MISO: track 159.4 -> 163.8 mm, vias 4 -> 8
- net EPD_BUSY: track 130.7 -> 134.7 mm, vias 5 -> 6
- net EPD_CS: track 190.2 -> 186.5 mm
- net EPD_RST: track 115.2 -> 118.8 mm, vias 5 -> 6
- net IO/BOOT: track 59.7 -> 62.5 mm
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